File: KICAD_PROJECT/GBS_SUPP_TOP/GBS_SUPP_TOP.kicad_pcb (KiCad board)
At the start: 2 copper layers, 116 x 100 mm, 27 parts, among them J1 CLK_PAD, J2 TO_GBS_I2C, J3 TO_GBS_CTL, J4 KEYPAD_IN, J5 KEYPAD_OUT, J6 I2C_OLED, J7 SIS351, J8 Encoder, J9 I2C_OLED, SW1 UP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

Commit message: Rev0.3A
Fix PLCC Board mounting hole problem.
Other:
- board text added: "for GBS8200 Rev 0.3A AUG/2021 (C) @Antarcticlion"
- board text removed: "for GBS8200 Rev 0.3 JUL/2021 (C) @Antarcticlion"
