File: KICAD_PROJECT/GBS_SUPP_TOP/GBS_SUPP_TOP.kicad_pcb (KiCad board)
At the start: 2 copper layers, 116 x 100 mm, 27 parts, among them J1 CLK_PAD, J2 TO_GBS_I2C, J3 TO_GBS_CTL, J4 KEYPAD_IN, J5 KEYPAD_OUT, J6 I2C_OLED, J7 SIS351, J8 Encoder, J9 I2C_OLED, SW1 UP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

Commit message: Rev 0.4
Support HD-VC9900
Parts:
- removed H5, H6: MountingHole, MountingHole:MountingHole_3.2mm_M3
- added H10: MountingHole, MountingHole:MountingHole_4.3mm_M4, F.Cu at (138.0, 9.00)
- added H11: MountingHole, MountingHole:MountingHole_4.3mm_M4, F.Cu at (138.0, 105.0)
- added H12: MountingHole, MountingHole:MountingHole_4.3mm_M4, F.Cu at (32.0, 9.00)
- added H13: MountingHole, MountingHole:MountingHole_4.3mm_M4, F.Cu at (107.0, 47.8)
- added H14: MountingHole, MountingHole:MountingHole_4.3mm_M4, F.Cu at (107.0, 86.2)
- added H15: MountingHole, MountingHole:MountingHole_4.3mm_M4, F.Cu at (131.0, 47.8)
- added H16: MountingHole, MountingHole:MountingHole_4.3mm_M4, F.Cu at (131.0, 86.2)
- added H9: MountingHole, MountingHole:MountingHole_4.3mm_M4, F.Cu at (32.0, 105.0)
- added J10: TO_GBS_UART, Connector_JST:JST_XH_B4B-XH-A_1x04_P2.50mm_Vertical, F.Cu at (96.8, 51.6)
- J3: value TO_GBS_CTL -> TO_GBS_CTL_LINE
- moved J5 86.5 mm to (114.0, 101.1)
- moved J4 15.5 mm to (114.0, 92.5)
- moved SW4 11.8 mm to (71.5, 19.8), turned to 0 degrees
- moved C2 11.5 mm to (75.1, 49.7)
- moved C1 11.5 mm to (67.7, 49.7)
- moved SW3 11.3 mm to (94.3, 19.8), turned to 0 degrees
- moved J2 9.81 mm to (86.7, 51.6)
- moved SW1 7.76 mm to (82.9, 30.0), turned to 0 degrees
- moved SW2 7.31 mm to (82.9, 19.8), turned to 0 degrees
- moved SW5 4.62 mm to (78.3, 38.9)
- moved J8 4.50 mm to (119.6, 6.90)
- moved J3 1.70 mm to (114.0, 25.0)
Connections:
- J3 pad 2: Net-(J3-Pad2) -> SCL
- J3 pad 3: Net-(J3-Pad3) -> SDA
Routing:
- net GND: track 0.00 -> 311.8 mm, vias 5 -> 0
- net SCL: track 127.8 -> 188.6 mm
- net SDA: track 139.3 -> 175.2 mm
- net UP: track 109.1 -> 93.7 mm
- net ENC_B: track 90.0 -> 104.3 mm
- net RIGHT: track 136.1 -> 122.2 mm
- net +3V3: track 150.2 -> 139.8 mm
- net DEBUG: track 51.3 -> 61.4 mm, vias 0 -> 1
- net ENC_SW: track 133.0 -> 128.2 mm
- net DOWN: track 122.2 -> 126.6 mm, vias 0 -> 1
- net ENC_A: track 87.4 -> 86.1 mm
- net LEFT: track 118.5 -> 117.3 mm
Other:
- board size 116 x 100 mm -> 116 x 106 mm
- board text added: "for GBS8200/8220/HD-VC9900 Rev 0.4 JUL/2021 (C) @Antarcticlion"
- board text removed: "for GBS8200 Rev 0.3A AUG/2021 (C) @Antarcticlion"

Commit message: Rev 0.6
Parts:
- removed J5: KEYPAD_OUT, Connector_JST:JST_XH_B5B-XH-A_1x05_P2.50mm_Vertical
- removed R1: 10KR, Resistor_THT:R_Axial_DIN0207_L6.3mm_D2.5mm_P10.16mm_Horizontal
- added J11: VGA_OUT, ryuk_lib:DB_15F-VGA_L, F.Cu at (55.0, 115.0)
- added J12: VGA_IN, Connector_JST:JST_PH_B12B-PH-K_1x12_P2.00mm_Vertical, B.Cu at (43.0, 92.0)
- added J20: TO_GBS_V5, Connector_JST:JST_XH_B6B-XH-A_1x06_P2.50mm_Vertical, F.Cu at (96.0, 56.0)
- added J6: I2C_OLED, Connector_JST:JST_XH_B4B-XH-A_1x04_P2.50mm_Vertical, F.Cu at (62.8, 20.7)
- added J9: I2C_OLED, Connector_JST:JST_XH_B4B-XH-A_1x04_P2.50mm_Vertical, F.Cu at (70.4, 40.0)
- J1: footprint Connector_JST:JST_XH_B3B-XH-A_1x03_P2.50mm_Vertical -> TerminalBlock_Phoenix:TerminalBlock_Phoenix_PTSM-0,5-3-2.5-H-THR_1x03_P2.50mm_Horizontal
- J7: value SIS351 -> SI5351_module
- moved SW4 90.7 mm to (112.0, 101.0)
- moved SW2 83.4 mm to (102.0, 101.0)
- moved SW3 81.2 mm to (92.0, 101.0)
- moved SW1 65.8 mm to (102.0, 93.0)
- moved J8 35.7 mm to (86.0, 19.0)
- moved SW5 19.1 mm to (97.0, 35.0)
- moved C2 17.8 mm to (82.9, 65.7)
- moved C1 17.8 mm to (75.5, 65.7)
- moved J10 13.3 mm to (84.0, 55.0)
- moved J2 13.1 mm to (74.0, 55.0)
- moved J6 6.00 mm to (36.8, 20.7)
- moved J9 6.00 mm to (44.4, 40.0)
- moved J1 5.59 mm to (37.1, 63.7)
- moved J7 5.59 mm to (48.2, 73.7)
- moved U2 5.59 mm to (51.9, 66.3)
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Routing:
- net SDA: track 175.2 -> 287.8 mm
- net DOWN: track 126.6 -> 20.8 mm, vias 1 -> 0
- net RIGHT: track 122.2 -> 21.4 mm
- net LEFT: track 117.3 -> 34.0 mm
- net UP: track 93.7 -> 14.1 mm
- net VGA_GND: track 0.00 -> 74.6 mm
- net GND: track 311.8 -> 383.1 mm
- net SCL: track 188.6 -> 236.7 mm
- net VGA_H: track 0.00 -> 45.1 mm
- net VGA_V: track 0.00 -> 23.6 mm
- net +3V3: track 139.8 -> 159.9 mm
- net ENC_B: track 104.3 -> 91.5 mm
- net VGA_R: track 0.00 -> 12.0 mm
- net VGA_G: track 0.00 -> 11.3 mm
- net VGA_B: track 0.00 -> 10.6 mm
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Other:
- outline, holes or cut-outs redrawn
- board text added: "GND"
- board text added: "VCC"
- board text added: "for GBS8200/8220/HD-VC9900 Rev 0.6 SEP/2021 (C) @Antarcticlion"
- board text removed: "for GBS8200/8220/HD-VC9900 Rev 0.4 JUL/2021 (C) @Antarcticlion"
